File: Electronics/2-Hardware/Burner.sch (KiCad schematic (older format))
At the start: 14 parts, among them P1 CONN_2, P2 CONN_2, P3 CONN_1, P4 CONN_2, P5 CONN_2, P6 CONN_1, Q1 DMN2230U-7, U1 LM317AEMP, U2 MSP430G2553-20, U3 ISL32612

Commit message: Started new design. Fixes #1, fixes #4, fixes #6.
Parts:
- removed P4: CONN_2, ~, symbol CONN_2
- removed R2: 2.7, ~, symbol R
- removed U1: LM317AEMP, ~, symbol LM317-4PIN
- added P?: CONN_4, ~, symbol CONN_4
- added R?: 1, ~, symbol R
- added R?: 1k, ~, symbol R
- added R? (x2): 10k, ~, symbol R
- added U?: DAC5311, symbol DAC5311
- added U? (x2): ADA4805-1, symbol ADA4805-1
Connections:
- net labels added: +12V, +3.3V, MOSI, OP_CTRL, SCLK, SENSE, SYNC
- net labels removed: MOS_TRIG, NI_Out
- wire segments 53 -> 95
Other:
- moved on the sheet: P3, P6, Q1, R1

Commit message: Added boost convertor to schematic
Parts:
- added Q?: MOS_P, ~, symbol MOS_P
- added R?: 10k, ~, symbol R
- added U?: LM3481, symbol LM3481
Connections:
- net +BATT: now also Q?.D; no longer P2.2 (PM)
- net GND: now also R?.2
- new net: P2.2 (PM), Q?.S
- new net: Q?.G, R?.1
Other:
- moved on the sheet: C1, C2, P1, P2, P5, P?, R?, U2, U3

Commit message: Changed DAC to be a LPF style
Parts:
- removed U?: DAC5311, symbol DAC5311
- added C? (x3): 0.1uF, ~, symbol C
- added R?: 1.6k, ~, symbol R
Connections:
- net +3.3V: now also C?.1, C?.1
- net GND: now also C?.2, C?.2, C?.2
- net PWM: now reaches U2.19 (P2.6)
- net PWM: now also R?.1
- net MOSI: no longer names the net of U2.15 (P1.7)
- net SCLK: no longer names the net of U2.7 (P1.5)
- net SYNC: no longer names the net of U2.6 (P1.4)
- new net: C?.1, R?.2, U?.~ (~SHUTDOWN)
Changed lines of the file:
@@
 Sheet 1 1
 Title ""
-Date "25 feb 2015"
+Date "28 feb 2015"
 Rev ""
 Comp ""
@@
 L GND #PWR05
 U 1 1 5301C4C1
-P 9050 3600
-F 0 "#PWR05" H 9050 3600 30  0001 C CNN
-F 1 "GND" H 9050 3530 30  0001 C CNN
-F 2 "" H 9050 3600 60  0000 C CNN
-F 3 "" H 9050 3600 60  0000 C CNN
-	1    9050 3600
+P 8950 3200
+F 0 "#PWR05" H 8950 3200 30  0001 C CNN
+F 1 "GND" H 8950 3130 30  0001 C CNN
+F 2 "" H 8950 3200 60  0000 C CNN
+F 3 "" H 8950 3200 60  0000 C CNN
+	1    8950 3200
 	1    0    0    -1
 $EndComp
 Wire Wire Line
 	8900 3550 9050 3550
-Wire Wire Line
-	9050 3150 9050 3600
 $Comp
 L R R1
@@
 	1    0    0    -1
 $EndComp
-Wire Wire Line
-	7900 4150 7650 4150
 $Comp
 L CONN_2 P1
@@
 Wire Wire Line
 	8600 3150 9050 3150
-Connection ~ 9050 3550
 $Comp
 L DIFF_RX U3
@@
 Wire Wire Line
 	3450 7100 3450 7050
-$Comp
-L DAC5311 U?
-U 1 1 54E43F1B
-P 1450 6250
-F 0 "U?" H 1700 6600 60  0000 C CNN
-F 1 "DAC5311" H 1650 5900 60  0000 C CNN
-F 2 "" H 1450 5700 60  0000 C CNN
-F 3 "" H 1450 5700 60  0000 C CNN
-	1    1450 6250
-	1    0    0    -1
-$EndComp
-Wire Wire Line
-	1850 6250 2350 6250
-$Comp
-L GND #PWR?
-U 1 1 54E43F7D
-P 1450 6700
-F 0 "#PWR?" H 1450 6700 30  0001 C CNN
-F 1 "GND" H 1450 6630 30  0001 C CNN
-F 2 "" H 1450 6700 60  0000 C CNN
-F 3 "" H 1450 6700 60  0000 C CNN
-	1    1450 6700
-	1    0    0    -1
-$EndComp
-$Comp
-L +3.3V #PWR?
-U 1 1 54E43F8C
-P 1450 5750
-F 0 "#PWR?" H 1450 5710 30  0001 C CNN
-F 1 "+3.3V" H 1450 5860 30  0000 C CNN
-F 2 "" H 1450 5750 60  0000 C CNN
-F 3 "" H 1450 5750 60  0000 C CNN
-	1    1450 5750
-	1    0    0    -1
-$EndComp
-Wire Wire Line
-	1450 5850 1450 5750
-Wire Wire Line
-	1450 6650 1450 6700
-Text Label 7650 4150 2    60   ~ 0
-SCLK
-Text Label 9000 4050 0    60   ~ 0
-MOSI
-Wire Wire Line
-	9000 4050 8900 4050
+Wire Wire Line
+	1550 6250 2350 6250
 $Comp
 L GND #PWR?
@@
 Wire Wire Line
 	8900 4150 9500 4150
-Text Label 900  6350 2    60   ~ 0
-MOSI
-Text Label 900  6250 2    60   ~ 0
-SCLK
-Wire Wire Line
-	1050 6350 900  6350
-Wire Wire Line
-	900  6250 1050 6250
-Text Label 7650 4050 2    60   ~ 0
-SYNC
-Wire Wire Line
-	7900 4050 7650 4050
-Text Label 900  6150 2    60   ~ 0
-SYNC
-Wire Wire Line
-	900  6150 1050 6150
 $Comp
 L ADA4805-1 U?
@@
 L +3.3V #PWR?
 U 1 1 54E45110
-P 5450 6600
-F 0 "#PWR?" H 5450 6560 30  0001 C CNN
-F 1 "+3.3V" H 5450 6710 30  0000 C CNN
-F 2 "" H 5450 6600 60  0000 C CNN
-F 3 "" H 5450 6600 60  0000 C CNN
-	1    5450 6600
-	1    0    0    -1
-$EndComp
-Wire Wire Line
-	5450 6650 5450 6600
+P 5450 6500
+F 0 "#PWR?" H 5450 6460 30  0001 C CNN
+F 1 "+3.3V" H 5450 6610 30  0000 C CNN
+F 2 "" H 5450 6500 60  0000 C CNN
+F 3 "" H 5450 6500 60  0000 C CNN
+	1    5450 6500
+	1    0    0    -1
+$EndComp
+Wire Wire Line
+	5450 6650 5450 6500
 Wire Wire Line
 	4850 7250 4850 7550
@@
 Wire Wire Line
 	2350 1000 2350 900
+$Comp
+L R R?
+U 1 1 54F16152
+P 1300 6250
+F 0 "R?" V 1380 6250 40  0000 C CNN
+F 1 "1.6k" V 1307 6251 40  0000 C CNN
+F 2 "~" V 1230 6250 30  0000 C CNN
+F 3 "~" H 1300 6250 30  0000 C CNN
+	1    1300 6250
+	0    -1   -1   0
+$EndComp
+$Comp
+L C C?
+U 1 1 54F16161
+P 1700 6550
+F 0 "C?" H 1700 6650 40  0000 L CNN
+F 1 "0.1uF" H 1706 6465 40  0000 L CNN
+F 2 "~" H 1738 6400 30  0000 C CNN
+F 3 "~" H 1700 6550 60  0000 C CNN
+	1    1700 6550
+	1    0    0    -1
+$EndComp
+Wire Wire Line
+	1700 6250 1700 6350
+Connection ~ 1700 6250
+$Comp
+L GND #PWR?
+U 1 1 54F16243
+P 1700 6800
+F 0 "#PWR?" H 1700 6800 30  0001 C CNN
+F 1 "GND" H 1700 6730 30  0001 C CNN
+F 2 "" H 1700 6800 60  0000 C CNN
+F 3 "" H 1700 6800 60  0000 C CNN
+	1    1700 6800
+	1    0    0    -1
+$EndComp
+Wire Wire Line
+	1700 6750 1700 6800
+Text Label 950  6250 2    60   ~ 0
+PWM
+Wire Wire Line
+	1050 6250 950  6250
+Text Label 9050 3650 0    60   ~ 0
+PWM
+Wire Wire Line
+	9050 3150 9050 3550
+Wire Wire Line
+	8950 3150 8950 3200
+Connection ~ 8950 3150
+Wire Wire Line
+	9050 3650 8900 3650
+$Comp
+L C C?
+U 1 1 54F16582
+P 3200 6100
+F 0 "C?" H 3200 6200 40  0000 L CNN
+F 1 "0.1uF" H 3206 6015 40  0000 L CNN
+F 2 "~" H 3238 5950 30  0000 C CNN
+F 3 "~" H 3200 6100 60  0000 C CNN
+	1    3200 6100
+	0    -1   -1   0
+$EndComp
+$Comp
+L GND #PWR?
+U 1 1 54F16591
+P 3500 6150
+F 0 "#PWR?" H 3500 6150 30  0001 C CNN
+F 1 "GND" H 3500 6080 30  0001 C CNN
+F 2 "" H 3500 6150 60  0000 C CNN
+F 3 "" H 3500 6150 60  0000 C CNN
+	1    3500 6150
+	1    0    0    -1
+$EndComp
+$Comp
+L GND #PWR?
+U 1 1 54F165A0
+P 6100 6650
+F 0 "#PWR?" H 6100 6650 30  0001 C CNN
+F 1 "GND" H 6100 6580 30  0001 C CNN
+F 2 "" H 6100 6650 60  0000 C CNN
+F 3 "" H 6100 6650 60  0000 C CNN
+	1    6100 6650
+	1    0    0    -1
+$EndComp
+$Comp
+L C C?
+U 1 1 54F165AF
+P 5850 6550
+F 0 "C?" H 5850 6650 40  0000 L CNN
+F 1 "0.1uF" H 5856 6465 40  0000 L CNN
+F 2 "~" H 5888 6400 30  0000 C CNN
+F 3 "~" H 5850 6550 60  0000 C CNN
+	1    5850 6550
+	0    -1   -1   0
+$EndComp
+Wire Wire Line
+	6050 6550 6100 6550
+Wire Wire Line
+	6100 6550 6100 6650
+Wire Wire Line
+	5650 6550 5450 6550
+Connection ~ 5450 6550
+Wire Wire Line
+	3400 6100 3500 6100
+Wire Wire Line
+	3500 6100 3500 6150
+Wire Wire Line
+	3000 6100 2750 6100
+Connection ~ 2750 6100
 $EndSCHEMATC
